Commit message: Added teleop to launch

File: src/my_robot/urdf/my_robot.xacro (robot description, xacro)
@@ -31,28 +31,4 @@
       </geometry>
     </visual>
-    <!--collision name='back_caster_collision'>
-      <origin xyz="-0.15 0 -0.05" rpy=" 0 0 0"/>
-      <geometry>
-        <sphere radius="0.0499"/>
-      </geometry>
-    </collision>
-    <visual name='back_caster_visual'>
-      <origin xyz="-0.15 0 -0.05" rpy=" 0 0 0"/>
-      <geometry>
-        <sphere radius="0.05"/>
-      </geometry>
-    </visual-->
-    <!--collision name='front_caster_collision'>
-      <origin xyz="0.15 0 -0.05" rpy=" 0 0 0"/>
-      <geometry>
-        <sphere radius="0.0499"/>
-      </geometry>
-    </collision>
-    <visual name='front_caster_visual'>
-      <origin xyz="0.15 0 -0.05" rpy=" 0 0 0"/>
-      <geometry>
-        <sphere radius="0.05"/>
-      </geometry>
-    </visual-->
   </link>
   <!--- 4 Wheels -->

Commit message: Updated robot structure and changed the dif drive plugin

File: src/my_robot/urdf/my_robot.xacro (robot description, xacro)
@@ -1,6 +1,6 @@
 <?xml version='1.0'?>
 <robot name="my_robot" xmlns:xacro="http://www.ros.org/wiki/xacro">
+  <link name="robot_footprint"></link>
   <xacro:include filename="$(find my_robot)/urdf/my_robot.gazebo" />
-  <link name="robot_footprint"></link>
   <joint name="robot_footprint_joint" type="fixed">
     <origin xyz="0 0 0" rpy="0 0 0" />
@@ -22,5 +22,5 @@
       <origin xyz="0 0 0" rpy=" 0 0 0"/>
       <geometry>
-        <box size=".4 .4 .1"/>
+        <box size=".4 .2 .1"/>
       </geometry>
     </collision>
@@ -31,23 +31,48 @@
       </geometry>
     </visual>
+    <collision name='back_caster_collision'>
+      <origin xyz="-0.15 0 -0.05" rpy=" 0 0 0"/>
+      <geometry>
+        <sphere radius="0.0499"/>
+      </geometry>
+    </collision>
+    <visual name='back_caster_visual'>
+      <origin xyz="-0.15 0 -0.05" rpy=" 0 0 0"/>
+      <geometry>
+        <sphere radius="0.05"/>
+      </geometry>
+    </visual>
+    <collision name='front_caster_collision'>
+      <origin xyz="0.15 0 -0.05" rpy=" 0 0 0"/>
+      <geometry>
+        <sphere radius="0.0499"/>
+      </geometry>
+    </collision>
+    <visual name='front_caster_visual'>
+      <origin xyz="0.15 0 -0.05" rpy=" 0 0 0"/>
+      <geometry>
+        <sphere radius="0.05"/>
+      </geometry>
+    </visual>
   </link>
-  <!--- 4 Wheels -->
-  <link name="left_wheel_back">
+  <link name='left_wheel'>
+    <pose>0 0 0 0 0 0</pose>
     <inertial>
-      <origin xyz="0 0 0" rpy="0 1.5707 1.5707"/>
-      <mass value="5"/>
+      <mass value="5.0"/>
+      <origin xyz="0.0 0 0" rpy=" 0 1.5707 1.5707"/>
       <inertia
-              ixx="0.1" ixy="0" ixz="0"
-              iyy="0.1" iyz="0" izz="0.1"
+          ixx="0.1" ixy="0" ixz="0"
+          iyy="0.1" iyz="0"
+          izz="0.1"
       />
     </inertial>
-    <collision>
-      <origin xyz="0 0 0" rpy="0 1.5707 1.5707"/>
+    <collision name='collision'>
+      <origin xyz="0 0 0" rpy=" 0 1.5707 1.5707"/>
       <geometry>
         <cylinder radius="0.1" length="0.05"/>
       </geometry>
     </collision>
-    <visual>
-      <origin xyz="0 0 0" rpy="0 1.5707 1.5707"/>
+    <visual name='left_wheel_visual'>
+      <origin xyz="0 0 0" rpy=" 0 1.5707 1.5707"/>
       <geometry>
         <cylinder radius="0.1" length="0.05"/>
@@ -55,7 +80,31 @@
     </visual>
   </link>
-  <joint name="left_wheel_back_hinge" type="continuous">
-    <origin xyz="-0.12 0.25 0" rpy="0 0 0"/>
-    <child link="left_wheel_back"/>
+  <link name='right_wheel'>
+    <pose>0 0 0 0 0 0</pose>
+    <inertial>
+      <mass value="5.0"/>
+      <origin xyz="0.0 0 0" rpy=" 0 1.5707 1.5707"/>
+      <inertia
+          ixx="0.1" ixy="0" ixz="0"
+          iyy="0.1" iyz="0"
+          izz="0.1"
+      />
+    </inertial>
+    <collision name='collision'>
+      <origin xyz="0 0 0" rpy=" 0 1.5707 1.5707"/>
+      <geometry>
+        <cylinder radius="0.1" length="0.05"/>
+      </geometry>
+    </collision>
+    <visual name='right_wheel_visual'>
+      <origin xyz="0 0 0" rpy=" 0 1.5707 1.5707"/>
+      <geometry>
+        <cylinder radius="0.1" length="0.05"/>
+      </geometry>
+    </visual>
+  </link>
+  <joint type="continuous" name="left_wheel_hinge">
+    <origin xyz="0 0.25 0" rpy="0 0 0"/>
+    <child link="left_wheel"/>
     <parent link="chassis"/>
     <axis xyz="0 1 0" rpy="0 0 0"/>
@@ -63,29 +112,7 @@
     <dynamics damping="1.0" friction="1.0"/>
   </joint>
-  <link name="left_wheel_front">
-    <inertial>
-      <origin xyz="0 0 0" rpy="0 1.5707 1.5707"/>
-      <mass value="5"/>
-      <inertia
-              ixx="0.1" ixy="0" ixz="0"
-              iyy="0.1" iyz="0" izz="0.1"
-      />
-    </inertial>
-    <collision>
-      <origin xyz="0 0 0" rpy="0 1.5707 1.5707"/>
-      <geometry>
-        <cylinder radius="0.1" length="0.05"/>
-      </geometry>
-    </collision>
-    <visual>
-      <origin xyz="0 0 0" rpy="0 1.5707 1.5707"/>
-      <geometry>
-        <cylinder radius="0.1" length="0.05"/>
-      </geometry>
-    </visual>
-  </link>
-  <joint name="left_wheel_front_hinge" type="continuous">
-    <origin xyz="0.12 0.25 0" rpy="0 0 0"/>
-    <child link="left_wheel_front"/>
+  <joint type="continuous" name="right_wheel_hinge">
+    <origin xyz="0 -0.25 0" rpy="0 0 0"/>
+    <child link="right_wheel"/>
     <parent link="chassis"/>
     <axis xyz="0 1 0" rpy="0 0 0"/>
@@ -93,29 +120,31 @@
     <dynamics damping="1.0" friction="1.0"/>
   </joint>
-  <link name="right_wheel_back">
+  <link name='camera'>
+    <pose>0 0 0 0 0 0</pose>
     <inertial>
-      <origin xyz="0 0 0" rpy="0 1.5707 1.5707"/>
-      <mass value="5"/>
+      <mass value="0.1"/>
+      <origin xyz="0.0 0 0" rpy="0.0 0 0"/>
       <inertia
-              ixx="0.1" ixy="0" ixz="0"
-              iyy="0.1" iyz="0" izz="0.1"
+          ixx="1e-6" ixy="0" ixz="0"
+          iyy="1e-6" iyz="0"
+          izz="1e-6"
       />
     </inertial>
-    <collision>
-      <origin xyz="0 0 0" rpy="0 1.5707 1.5707"/>
+    <collision name='collision'>
+      <origin xyz="0 0 0" rpy=" 0 0 0"/>
       <geometry>
-        <cylinder radius="0.1" length="0.05"/>
+        <box size="0.05 0.05 0.05"/>
       </geometry>
     </collision>
-    <visual>
-      <origin xyz="0 0 0" rpy="0 1.5707 1.5707"/>
+    <visual name='camera_visual'>
+      <origin xyz="0 0 0" rpy="0 0 0"/>
       <geometry>
-        <cylinder radius="0.1" length="0.05"/>
+        <box size="0.05 0.05 0.05"/>
       </geometry>
     </visual>
   </link>
-  <joint name="right_wheel_back_hinge" type="continuous">
-    <origin xyz="-0.12 -0.25 0" rpy="0 0 0"/>
-    <child link="right_wheel_back"/>
+  <joint type="fixed" name="camera_joint">
+    <origin xyz="0.2 0 0" rpy="0 0 0"/>
+    <child link="camera"/>
     <parent link="chassis"/>
     <axis xyz="0 1 0" rpy="0 0 0"/>
@@ -123,29 +152,31 @@
     <dynamics damping="1.0" friction="1.0"/>
   </joint>
-  <link name="right_wheel_front">
+  <link name='hokuyo'>
+    <pose>0 0 0 0 0 0</pose>
     <inertial>
-      <origin xyz="0 0 0" rpy="0 1.5707 1.5707"/>
-      <mass value="5"/>
+      <mass value="1e-5"/>
+      <origin xyz="0.0 0 0" rpy="0.0 0 0"/>
       <inertia
-              ixx="0.1" ixy="0" ixz="0"
-              iyy="0.1" iyz="0" izz="0.1"
+          ixx="1e-6" ixy="0" ixz="0"
+          iyy="1e-6" iyz="0"
+          izz="1e-6"
       />
     </inertial>
-    <collision>
-      <origin xyz="0 0 0" rpy="0 1.5707 1.5707"/>
+    <collision name='collision'>
+      <origin xyz="0 0 0" rpy=" 0 0 0"/>
       <geometry>
-        <cylinder radius="0.1" length="0.05"/>
+        <box size="0.1 0.1 0.1"/>
       </geometry>
     </collision>
-    <visual>
-      <origin xyz="0 0 0" rpy="0 1.5707 1.5707"/>
+    <visual name='hokuyo_visual'>
+      <origin xyz="0 0 0" rpy="0 0 0"/>
       <geometry>
-        <cylinder radius="0.1" length="0.05"/>
+        <mesh filename="package://my_robot/meshes/hokuyo.dae"/>
       </geometry>
     </visual>
   </link>
-  <joint name="right_wheel_front_hinge" type="continuous">
-    <origin xyz="0.12 -0.25 0" rpy="0 0 0"/>
-    <child link="right_wheel_front"/>
+  <joint type="fixed" name="hokuyo_joint">
+    <origin xyz="0.15 0.0 0.1" rpy="0 0 0"/>
+    <child link="hokuyo"/>
     <parent link="chassis"/>
     <axis xyz="0 1 0" rpy="0 0 0"/>
@@ -153,75 +184,3 @@
     <dynamics damping="1.0" friction="1.0"/>
   </joint>
-  <!--- Camera -->
-  <link name="camera">
-    <inertial>
-      <origin xyz="0 0 0" rpy="0 0 0"/>
-      <mass value="0.1"/>
-      <inertia
-              ixx="1e-6" ixy="0" ixz="0"
-              iyy="1e-6" iyz="0" izz="1e-6"
-      />
-    </inertial>
-    <collision>
-      <geometry>
-        <box size="0.05 0.05 0.05"/>
-      </geometry>
-    </collision>
-    <visual>
-      <geometry>
-        <box size="0.05 0.05 0.05"/>
-      </geometry>
-    </visual>
-  </link>
-  <joint name="camera_joint" type="fixed">
-    <origin xyz="0.2 0 0" rpy="0 0 0"/>
-    <child link="camera"/>
-    <parent link="chassis"/>
-    <axis xyz="0 1 0"/>
-  </joint>
-  <!--- LiDAR -->
-  <link name="hokuyo">
-    <inertial>
-      <origin xyz="0 0 0" rpy="0 0 0"/>
-      <mass value="1e-5"/>
-      <inertia
-              ixx="1e-6" ixy="0" ixz="0"
-              iyy="1e-6" iyz="0" izz="1e-6"
-      />
-    </inertial>
-    <collision>
-      <geometry>
-        <box size="0.1 0.1 0.1"/>
-      </geometry>
-    </collision>
-    <visual>
-      <geometry>
-        <mesh filename = "package://my_robot/meshes/hokuyo.dae"/>
-      </geometry>
-    </visual>
-  </link>
-  <joint name="hokuyo_joint" type="fixed">
-    <origin xyz="0.15 0 0.1" rpy="0 0 0"/>
-    <child link="hokuyo"/>
-    <parent link="chassis"/>
-    <axis xyz="0 1 0"/>
-  </joint>
-  <gazebo reference="camera">
-    <material>Gazebo/Red</material>
-  </gazebo>
-  <gazebo reference="chassis">
-    <material>Gazebo/SkyBlue</material>
-  </gazebo>
-  <gazebo reference="left_wheel_back">
-    <material>Gazebo/DarkYellow</material>
-  </gazebo>
-  <gazebo reference="left_wheel_front">
-    <material>Gazebo/DarkYellow</material>
-  </gazebo>
-  <gazebo reference="right_wheel_back">
-    <material>Gazebo/DarkYellow</material>
-  </gazebo>
-  <gazebo reference="right_wheel_front">
-    <material>Gazebo/DarkYellow</material>
-  </gazebo>
 </robot>

Commit message: mapping with rgb-d camera working

File: src/my_robot/urdf/my_robot.xacro (robot description, xacro)
@@ -152,4 +152,11 @@
     <dynamics damping="1.0" friction="1.0"/>
   </joint>
+  <joint name="camera_optical_joint" type="fixed">
+    <origin xyz="0 0 0" rpy="-1.5707 0 -1.5707"/>
+    <parent link="camera"/>
+    <child link="camera_link_optical"/>
+  </joint>
+  <link name="camera_link_optical">
+  </link>
   <link name='hokuyo'>
     <pose>0 0 0 0 0 0</pose>

Commit message: removed slam_gmap

File: src/my_robot/urdf/my_robot.xacro (robot description, xacro)
@@ -22,5 +22,5 @@
       <origin xyz="0 0 0" rpy=" 0 0 0"/>
       <geometry>
-        <box size=".4 .2 .1"/>
+        <box size=".3 .5 .1"/>
       </geometry>
     </collision>
@@ -28,5 +28,5 @@
       <origin xyz="0 0 0" rpy=" 0 0 0"/>
       <geometry>
-        <box size=".4 .4 .1"/>
+        <box size=".3 .5 .1"/>
       </geometry>
     </visual>
@@ -34,5 +34,5 @@
       <origin xyz="-0.15 0 -0.05" rpy=" 0 0 0"/>
       <geometry>
-        <sphere radius="0.0499"/>
+        <sphere radius="0.048"/>
       </geometry>
     </collision>
@@ -40,5 +40,5 @@
       <origin xyz="-0.15 0 -0.05" rpy=" 0 0 0"/>
       <geometry>
-        <sphere radius="0.05"/>
+        <sphere radius="0.048"/>
       </geometry>
     </visual>
@@ -46,5 +46,5 @@
       <origin xyz="0.15 0 -0.05" rpy=" 0 0 0"/>
       <geometry>
-        <sphere radius="0.0499"/>
+        <sphere radius="0.048"/>
       </geometry>
     </collision>
@@ -52,5 +52,5 @@
       <origin xyz="0.15 0 -0.05" rpy=" 0 0 0"/>
       <geometry>
-        <sphere radius="0.05"/>
+        <sphere radius="0.048"/>
       </geometry>
     </visual>
@@ -105,5 +105,5 @@
   </link>
   <joint type="continuous" name="left_wheel_hinge">
-    <origin xyz="0 0.25 0" rpy="0 0 0"/>
+    <origin xyz="0 0.3 0" rpy="0 0 0"/>
     <child link="left_wheel"/>
     <parent link="chassis"/>
@@ -113,5 +113,5 @@
   </joint>
   <joint type="continuous" name="right_wheel_hinge">
-    <origin xyz="0 -0.25 0" rpy="0 0 0"/>
+    <origin xyz="0 -0.3 0" rpy="0 0 0"/>
     <child link="right_wheel"/>
     <parent link="chassis"/>
@@ -145,5 +145,5 @@
   </link>
   <joint type="fixed" name="camera_joint">
-    <origin xyz="0.2 0 0" rpy="0 0 0"/>
+    <origin xyz="0.15 0 0.03" rpy="0 0 0"/>
     <child link="camera"/>
     <parent link="chassis"/>
@@ -184,5 +184,5 @@
   </link>
   <joint type="fixed" name="hokuyo_joint">
-    <origin xyz="0.15 0.0 0.1" rpy="0 0 0"/>
+    <origin xyz="0.125 0.0 0.08" rpy="0 0 0"/>
     <child link="hokuyo"/>
     <parent link="chassis"/>
